File: KiCAD_files/Shield_Nucleo.kicad_pcb (KiCad board)
At the start: 4 copper layers, 100 x 100 mm, 126 parts, among them J1 Conn_01x02, J2 RJ45_LED_Shielded, J3 RJ45_LED_Shielded, J4 Conn_01x03_Male, J5 Conn_01x05_Male, J6 Conn_01x02, J7 Power, J8 Conn_02x07_Odd_Even, SW1 SW_Push, U1 STM32G474RE, U2 AT25xxx, U3 TCAN334GDR, U4 AP1117-33, U5 UCC21222DR, U6 UCC21222DR, U7 SFH617A-2X009T, U8 RFM-0505s, U9 RFM-0505s, Y1 NX3225SA-16.000000MHZ-T1

Commit message: Add two new folders, Power and ShieldNucleo Definition Package. Add a drill map dimension on Kicad PCB for Power and ShieldNucleo. Change the colour of title block and add new logo on Power and ShieldNucleo scheme board.
Parts:
- C15, C16: value CP1_Small -> 47uF
- C29: value 10 to 47uF -> 10uF
- D1, D2: value RBR2MM60BTFTR -> RBR2MM60ATFTR
- FB1: value Ferrite_Bead_Small -> 100Ohm @ 100MHz
- U9: value RFM-0505s -> CME0512S3C
- Y1: value NX3225SA-16.000000MHZ-T1 -> ECS-240-10-33-AGM-TR - 24MHz
- moved BT1 11.5 mm to (128.2, 98.7)
- moved J1 11.5 mm to (134.4, 132.4)
- moved C29 11.5 mm to (85.0, 131.3)
- moved C36 11.5 mm to (111.3, 64.4)
- moved R19 11.5 mm to (128.4, 72.0)
- moved U5 11.5 mm to (93.1, 67.1)
- moved U9 11.5 mm to (107.9, 71.4)
- moved U3 11.5 mm to (64.3, 72.8)
- moved C1 11.5 mm to (106.7, 87.3)
- moved C10 11.5 mm to (90.0, 99.3)
- moved C11 11.5 mm to (92.5, 71.8)
- moved C12 11.5 mm to (103.0, 96.5)
- moved C13 11.5 mm to (99.3, 70.5)
- moved C14 11.5 mm to (100.4, 94.9)
- moved C17 11.5 mm to (85.8, 74.9)
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